File: PIM_V01/PIM_V01.kicad_pcb (KiCad board)
At the start: 4 copper layers, 93.3 x 61.7 mm, 252 parts, among them J1 Conn_01x06, J10 Conn_02x08_Odd_Even, J11 Conn_01x02, J12 Conn_01x02, J13 Conn_01x02, J4 USB_C_Receptacle_USB2.0_14P, J5 Conn_01x04, J6 Conn_01x04, J7 Conn_02x03_Odd_Even, J8 Conn_01x02, J9 Conn_02x08_Odd_Even, Q1 SQJ407EP-T1_GE3, Q2 PMOS, Q3 PMOS, Q4 NMOS, SW1 SW_Push, U1 TPS259541DSGR, U10 TPS62933, U11 AP2112K-3.3, U12 MP28167GQ-A-P, U13 MT29F1G01ABAFDWB-IT_F, U14 MB85RS256B, U2 USBLC6-2SC6, U3 STM32H7A3VITx, U4 MCP2562FDT-E/SN, U5 MCP2562FDT-E/SN, U6 TPS62933, U7 TPS62933, U8 TPS62933, U9 TPS62933, Y1 Crystal_GND24_Small

Commit message: V01 RELEASE. Gerbers created to order RAW PCB
Parts:
- added C105: 10nF, Capacitor_SMD:C_0603_1608Metric, F.Cu at (94.6, 58.6)
- added C106: 10nF, Capacitor_SMD:C_0603_1608Metric, F.Cu at (173.1, 57.8)
- added C107: 10nF, Capacitor_SMD:C_0603_1608Metric, F.Cu at (95.3, 115.4)
- added C108: 10nF, Capacitor_SMD:C_0603_1608Metric, F.Cu at (172.5, 115.5)
- added R83: 0R, Resistor_SMD:R_0603_1608Metric, F.Cu at (94.7, 60.2)
- added R84: 0R, Resistor_SMD:R_0603_1608Metric, F.Cu at (173.0, 59.3)
- added R85: 0R, Resistor_SMD:R_0603_1608Metric, F.Cu at (95.3, 113.9)
- added R86: 0R, Resistor_SMD:R_0603_1608Metric, F.Cu at (172.5, 114.0)
- H1, H2, H3, H4: value MountingHole -> MountingHole_Pad; footprint MountingHole:MountingHole_2.2mm_M2 -> MountingHole:MountingHole_2.2mm_M2_Pad
- J11, J12, J13: moved to F.Cu
- moved H4 349.0 mm to (176.9, 115.0)
- moved H2 348.9 mm to (177.0, 59.0)
- moved J10 347.7 mm to (175.4, 63.3)
- moved J12 347.6 mm to (169.1, 106.8), turned to 0 degrees
- moved C1 347.6 mm to (136.0, 104.4)
- moved C100 347.6 mm to (151.0, 83.9)
- moved C101 347.6 mm to (163.6, 69.0)
- moved C102 347.6 mm to (165.1, 69.0)
- moved C103 347.6 mm to (152.2, 63.7)
- moved C104 347.6 mm to (153.7, 63.7)
- moved C13 347.6 mm to (120.9, 106.9)
- moved C15 347.6 mm to (115.4, 102.7)
- moved C16 347.6 mm to (113.9, 90.7)
- moved C18 347.6 mm to (111.4, 93.5)
- moved C19 347.6 mm to (111.4, 105.5)
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Routing:
- net Net-(C106-Pad1): track 0.00 -> 7.07 mm
- net /nCRESET_FPGA: track 28.8 -> 22.1 mm
- net Net-(C107-Pad1): track 0.00 -> 6.35 mm
- net Net-(C105-Pad1): track 0.00 -> 5.61 mm
- net Net-(C108-Pad1): track 0.00 -> 5.44 mm
- net GND: track 20.4 -> 23.7 mm, vias 64 -> 479
- net /USART3_TX_PL: track 61.4 -> 59.1 mm
- net /I2C2_SCL_PL: track 58.1 -> 59.4 mm
- net /CDONE_FPGA: track 34.4 -> 35.1 mm
- net /+VARI_EN: track 29.5 -> 30.2 mm
- net /USART3_RX_PL: track 55.0 -> 55.5 mm
- net /SPI2_nCS_PL: track 44.8 -> 45.3 mm
Other:
- board size 93.3 x 61.7 mm -> 93 x 62 mm

Commit message: updated some of the 3D bodies, and updated the BRINGUP plan with results from the first attempt at population; many components were not made in the order, so am now blocked waiting for those.
Parts:
- C69: value 22uF -> 22uF 25V
- D1: value SMBJ13A -> SMBJ12A
- D13: value SMAJ13A -> SMBJ12A
- J1: footprint Connector_Molex:Molex_Pico-Lock_504050-0691_1x06-1MP_P1.50mm_Horizontal -> CustomFootprints:Molex_Pico-Lock_504050-0691_1x06-1MP_P1.50mm_Horizontal
- J4: footprint Connector_USB:USB_C_Receptacle_HCTL_HC-TYPE-C-16P-01A -> Connector_USB:USB_C_Receptacle_GCT_USB4105-xx-A_16P_TopMnt_Horizontal
