File: PIM_V01/PIM_V01.kicad_pcb (KiCad board)
At the start: 4 copper layers, 93 x 62 mm, 260 parts, among them J1 Conn_01x06, J10 Conn_02x08_Odd_Even, J11 Conn_01x02, J12 Conn_01x02, J13 Conn_01x02, J4 USB_C_Receptacle_USB2.0_14P, J5 Conn_01x04, J6 Conn_01x04, J7 Conn_02x03_Odd_Even, J8 Conn_01x02, J9 Conn_02x08_Odd_Even, Q1 SQJ407EP-T1_GE3, Q2 PMOS, Q3 PMOS, Q4 NMOS, SW1 SW_Push, U1 TPS259541DSGR, U10 TPS62933, U11 AP2112K-3.3, U12 MP28167GQ-A-P, U13 MT29F1G01ABAFDWB-IT_F, U14 MB85RS256B, U2 USBLC6-2SC6, U3 STM32H7A3VITx, U4 MCP2562FDT-E/SN, U5 MCP2562FDT-E/SN, U6 TPS62933, U7 TPS62933, U8 TPS62933, U9 TPS62933, Y1 Crystal_GND24_Small

Commit message: finished uploading all of the correct footprints and 3D bodies. this is now done, and barely different than what was fabricated - used all manufacturers FPs (instead of kicads), but this didn't cause any of the original connections to break. I will now start on V02 (incl FPGA and smaller)
Parts:
- C1, C104, C72, C78, C79, C8, C80, C95, C99: value 1uF -> C_Small
- C10, C11, C14, C15, C94: value 4.7uF -> C_Small
- C100, C64: value 27pF -> C_Small
- C101, C102, C43, C44, C45, C46, C47, C48, C59, C60, C61, C62, C76, C77: value 22uF -> C_Small
- C103, C12, C13, C16, C17, C2, C34, C35, C36, C40, C41, C42, C53, C54, C57, C58, C70, C73, C74, C81, C83, C84, C85, C86, C87, C88, C89, C90, C91, C92, C93, C98: value 0.1uF -> C_Small
- C105, C106, C107, C108, C38, C55, C56, C65, C66, C67: value 10nF -> C_Small
- C18, C19, C20, C21, C22, C23, C24, C25: value 47pF -> C_Small
- C26, C27: value 4.7nF -> C_Small
- C28, C29, C30, C31, C32, C33, C49, C50, C51, C52, C6, C7, C82, C9: value 10uF -> C_Small
- C3: value 3.3nF -> C_Small
- C37, C39: value 33nF -> C_Small
- C4, C5: value 47uF -> C_Small
- C63: value 100nF -> C_Small
- C68, C75: value 100uF -> C_Small
- C69: value 22uF 25V -> C_Small
- C71: value 22nF -> C_Small
- C96, C97: value 2.2uF -> C_Small
- D1: footprint CustomFootprints:SMBJ16A -> CustomFootprints:SMBJ12A
- D13: footprint Diode_SMD:D_SMA -> CustomFootprints:SMBJ12A
- D3: value PMEG4010 -> D_Schottky
- D4: value BZT52C15 -> D_Zener
- FL1, FL2: value Choke_CommonMode_FerriteCore_1243 -> ACT45B-101-2P-TL003; footprint Inductor_SMD:L_CommonModeChoke_Coilcraft_1812CAN -> CustomFootprints:ACT45B-101-2P-TL003_TDK
- L1, L2, L3, L4, L5: value 6.8uH -> L_Small
- L6: value 4.7uH -> L_Small
- R1, R4: value 5k1R -> R_Small
- R10, R11, R16, R17, R22, R23, R24, R35, R36, R74, R75, R76, R77, R78, R83, R84, R85, R86, R9: value 0R -> R_Small
- R12, R69: value 1MR -> R_Small
- R13, R14, R15, R26, R28, R30, R38, R40, R59, R60, R61, R66, R67, R7: value 10kR -> R_Small
- R18, R19, R20, R21: value 60R -> R_Small
- R2: value 866kR -> R_Small
- R25, R37: value 52.3kR -> R_Small
- R27, R39: value 31.6kR -> R_Small
- R29: value 4.99kR -> R_Small
- R3: value 150kR -> R_Small
- R31, R33, R6: value 470R -> R_Small
- R32, R34, R81, R82: value 100R -> R_Small
- R41, R42, R43, R44: value 1kR -> R_Small
- R45, R47, R49: value 470kR -> R_Small
- R46, R48, R50, R68, R70, R71, R72, R73, R8: value 100kR -> R_Small
- R5: value 511R -> R_Small
- R51, R52, R57, R58: value 4.7kR -> R_Small
- R53: value 430kR -> R_Small
- R54: value 400kR -> R_Small
- R55: value 21.5kR -> R_Small
- R56: value 43.2kR -> R_Small
- R62, R63, R64, R65: value 33R -> R_Small
- R79, R80: value 1.8kR -> R_Small
- U12: footprint CustomFootprints:QFN-16_MP28167_MNP -> CustomFootprints:MP28167GQ-A-P
- U13: value MT29F1G01ABAFDWB-IT_F -> GD5F1GQ5UEYIGR; footprint Package_SON:WSON-8-1EP_8x6mm_P1.27mm_EP3.4x4.3mm -> CustomFootprints:GD5F1GQ5UEYIGR
- moved D13 0.53 mm to (133.0, 106.5)
- moved FL2 0.30 mm to (107.6, 107.0), turned to 180 degrees
- moved FL1 0.20 mm to (107.7, 95.0), turned to 180 degrees
Connections:
- FL1 pad 1: /CAN/CAN0_RAW_N -> /CAN/CAN0_RAW_P
- FL1 pad 2: /CAN0_N -> /CAN/CAN0_RAW_N
- FL1 pad 3: /CAN0_P -> /CAN0_N
- FL1 pad 4: /CAN/CAN0_RAW_P -> /CAN0_P
- FL2 pad 1: /CAN/CAN1_RAW_N -> /CAN/CAN1_RAW_P
- FL2 pad 2: /CAN1_N -> /CAN/CAN1_RAW_N
- FL2 pad 3: /CAN1_P -> /CAN1_N
- FL2 pad 4: /CAN/CAN1_RAW_P -> /CAN1_P
- U13 pad 9: (no net) -> GND
Routing:
- net GND: vias 479 -> 478
- net +12V_HK: vias 30 -> 29
