File: PIM_V01/PIM_V01.kicad_sch (KiCad schematic)
At the start: 106 parts, among them J1 Conn_01x06, J10 Conn_02x08_Odd_Even, J4 USB_C_Receptacle_USB2.0_14P, J5 Conn_01x04, J6 Conn_01x04, J7 Conn_02x03_Odd_Even, J8 Conn_01x02, J9 Conn_02x08_Odd_Even, Q1 SQJ407EP-T1_GE3, Q2 PMOS, Q3 PMOS, Q4 NMOS, SW1 SW_Push, U1 TPS259541DSGR, U11 AP2112K-3.3, U13 GD5F1GQ5UEYIGR, U14 MB85RS256B, U2 USBLC6-2SC6, U3 STM32H7A3VITx, Y1 Crystal_GND24_Small

Commit message: somehow last push my components had lost their values, and only displayed their Kicad value, but I fixed that now
Parts:
- removed D1, D13: SMBJ12A, CustomFootprints:SMBJ12A, symbol Custom_Components:SMBJ12A
- removed U13: GD5F1GQ5UEYIGR, CustomFootprints:GD5F1GQ5UEYIGR, symbol Custom_Components:GD5F1GQ5UEYIGR
- added D1: SMBJ12A, CustomFootprints:SMBJ16A, symbol Device:D_Zener
- added D13: SMBJ12A, Diode_SMD:D_SMA, symbol Diode:SMAJ13A
- added U13: MT29F1G01ABAFDWB-IT_F, MT29F1G01ABAFDWB-IT_F:SON127P600X800X65-8N, symbol Custom_Components:MT29F1G01ABAFDWB-IT_F
- C1, C104, C78, C79, C8, C80, C95, C99: value C_Small -> 1uF
- C100, C64: value C_Small -> 27pF
- C103, C2, C81, C89, C90, C91, C92, C93, C98: value C_Small -> 0.1uF
- C105, C106, C107, C108: value C_Small -> 10nF
- C3: value C_Small -> 3.3nF
- C4, C5: value C_Small -> 47uF
- C6, C7, C82, C9: value C_Small -> 10uF
- C63: value C_Small -> 100nF
- C94: value C_Small -> 4.7uF
- C96, C97: value C_Small -> 2.2uF
- D3: value D_Schottky -> PMEG4010
- D4: value D_Zener -> BZT52C15
- Q1: footprint CustomFootprints:PowerPAK-SO-8L_Option-2_VIS -> PowerPAK-SO-8L_Option-2_VIS
- R1, R4: value R_Small -> 5k1R
- R11, R83, R84, R85, R86: value R_Small -> 0R
- R12, R69: value R_Small -> 1MR
- R13, R59, R60, R61, R66, R67, R7: value R_Small -> 10kR
- R2: value R_Small -> 866kR
- R3: value R_Small -> 150kR
- R5: value R_Small -> 511R
- R51, R52, R57, R58: value R_Small -> 4.7kR
- R6: value R_Small -> 470R
- R62, R63, R64, R65: value R_Small -> 33R
- R68, R70, R8: value R_Small -> 100kR
- R79, R80: value R_Small -> 1.8kR
- R81, R82: value R_Small -> 100R
- U1: footprint CustomFootprints:DSG0008A -> DSG0008A
Connections:
- net +12V_HK: now also D13.1 (A1)
- net +12V_IN: now also D1.1 (K)
- net +3V3_MCU: now also U13.8 (VCC)
- net GND: now also D1.2 (A), D13.2 (A2), U13.4 (VSS)
- net OCTOSPI1_BK2_IO0: now also U13.5 (SI/IO0)
- net OCTOSPI1_BK2_IO1: now also U13.2 (SO/IO1)
- net OCTOSPI1_BK2_IO2: now also U13.3 (WP#/IO2)
- net OCTOSPI1_BK2_IO3: now also U13.7 (HOLD#/IO3)
- net OCTOSPI1_BK2_NCS: now also U13.1 (CS#)
- net OCTOSPI1_CLK: now also U13.6 (SCK)
Other:
- moved on the sheet: C80, C81

Commit message: finished uploading all of the correct footprints and 3D bodies. this is now done, and barely different than what was fabricated - used all manufacturers FPs (instead of kicads), but this didn't cause any of the original connections to break. I will now start on V02 (incl FPGA and smaller)
Parts:
- removed D1: SMBJ12A, CustomFootprints:SMBJ16A, symbol Device:D_Zener
- removed D13: SMBJ12A, Diode_SMD:D_SMA, symbol Diode:SMAJ13A
- removed U13: MT29F1G01ABAFDWB-IT_F, MT29F1G01ABAFDWB-IT_F:SON127P600X800X65-8N, symbol Custom_Components:MT29F1G01ABAFDWB-IT_F
- added D1, D13: SMBJ12A, CustomFootprints:SMBJ12A, symbol Custom_Components:SMBJ12A
- added U13: GD5F1GQ5UEYIGR, CustomFootprints:GD5F1GQ5UEYIGR, symbol Custom_Components:GD5F1GQ5UEYIGR
- C1, C104, C78, C79, C8, C80, C95, C99: value 1uF -> C_Small
- C100, C64: value 27pF -> C_Small
- C103, C2, C81, C89, C90, C91, C92, C93, C98: value 0.1uF -> C_Small
- C105, C106, C107, C108: value 10nF -> C_Small
- C3: value 3.3nF -> C_Small
- C4, C5: value 47uF -> C_Small
- C6, C7, C82, C9: value 10uF -> C_Small
- C63: value 100nF -> C_Small
- C94: value 4.7uF -> C_Small
- C96, C97: value 2.2uF -> C_Small
- D3: value PMEG4010 -> D_Schottky
- D4: value BZT52C15 -> D_Zener
- Q1: footprint PowerPAK-SO-8L_Option-2_VIS -> CustomFootprints:PowerPAK-SO-8L_Option-2_VIS
- R1, R4: value 5k1R -> R_Small
- R11, R83, R84, R85, R86: value 0R -> R_Small
- R12, R69: value 1MR -> R_Small
- R13, R59, R60, R61, R66, R67, R7: value 10kR -> R_Small
- R2: value 866kR -> R_Small
- R3: value 150kR -> R_Small
- R5: value 511R -> R_Small
- R51, R52, R57, R58: value 4.7kR -> R_Small
- R6: value 470R -> R_Small
- R62, R63, R64, R65: value 33R -> R_Small
- R68, R70, R8: value 100kR -> R_Small
- R79, R80: value 1.8kR -> R_Small
- R81, R82: value 100R -> R_Small
- U1: footprint DSG0008A -> CustomFootprints:DSG0008A
Connections:
- net +12V_HK: now also D13.1
- net +12V_IN: now also D1.1
- net +3V3_MCU: now also U13.8 (VCC)
- net GND: now also D1.2, D13.2, U13.4 (VSS), U13.9 (EP)
- net OCTOSPI1_BK2_IO0: now also U13.5 (SI/SIO0)
- net OCTOSPI1_BK2_IO1: now also U13.2 (SO/SIO1)
- net OCTOSPI1_BK2_IO2: now also U13.3 (WP#/SIO2)
- net OCTOSPI1_BK2_IO3: now also U13.7 (HOLD#/SIO3)
- net OCTOSPI1_BK2_NCS: now also U13.1 (CS#)
- net OCTOSPI1_CLK: now also U13.6 (SCLK)
Other:
- moved on the sheet: C80, C81
