File: PIM_V01/PIM_V01.kicad_sch (KiCad schematic)
At the start: 98 parts, among them J1 Conn_01x06, J10 Conn_02x08_Odd_Even, J4 USB_C_Receptacle_USB2.0_14P, J5 Conn_01x04, J6 Conn_01x04, J7 Conn_02x03_Odd_Even, J8 Conn_01x02, J9 Conn_02x08_Odd_Even, Q1 SQJ407EP-T1_GE3, Q2 PMOS, Q3 PMOS, Q4 NMOS, SW1 SW_Push, U1 TPS259541DSGR, U11 AP2112K-3.3, U13 MT29F1G01ABAFDWB-IT_F, U14 MB85RS256B, U2 USBLC6-2SC6, U3 STM32H7A3VITx, Y1 Crystal_GND24_Small

Commit message: V01 RELEASE. Gerbers created to order RAW PCB
Parts:
- removed H1, H2, H3, H4: MountingHole, MountingHole:MountingHole_2.2mm_M2, symbol Mechanical:MountingHole
- added C105, C106, C107, C108: 10nF, Capacitor_SMD:C_0603_1608Metric, symbol Device:C_Small
- added H1, H2, H3, H4: MountingHole_Pad, MountingHole:MountingHole_2.2mm_M2_Pad, symbol Mechanical:MountingHole_Pad
- added R83, R84, R85, R86: 0R, Resistor_SMD:R_0603_1608Metric, symbol Device:R_Small
Connections:
- net GND: now also C105.2, C106.2, C107.2, C108.2, R83.2, R84.2, R85.2, R86.2
- new net: C107.1, H3.1, R85.1
- new net: C106.1, H2.1, R84.1
- new net: C105.1, H1.1, R83.1
- new net: C108.1, H4.1, R86.1
Other:
- moved on the sheet: J7

Commit message: updated some of the 3D bodies, and updated the BRINGUP plan with results from the first attempt at population; many components were not made in the order, so am now blocked waiting for those.
Parts:
- C1: MD (none) -> CAP CER 1UF 25V X7R 0603; MPN (none) -> GCM188R71E105KA64J; PD (none) -> CAP CER 1UF 25V X7R 0603
- C100, C64: MPN (none) -> GCM1885C1H270JA16D; PD (none) -> CAP CER 27PF 50V C0G/NP0 0603
- C103, C2, C63, C81, C89, C90, C91, C92, C93, C98: MPN (none) -> GCM188R71H104KA57D; PD (none) -> CAP CER 0.1UF 50V X7R 0603
- C104, C78, C79, C8, C80, C95, C99: MPN (none) -> GCM188R71E105KA64J; PD (none) -> CAP CER 1UF 25V X7R 0603
- C105, C106, C107, C108: MPN (none) -> GCM188R71H103KA37J; PD (none) -> CAP CER 10000PF 50V X7R 0603
- C3: MPN (none) -> GCM1885C1H332JA16D; PD (none) -> CAP CER 3300PF 50V C0G/NP0 0603
- C4, C5: MPN (none) -> GRT188R61E106ME13D; Note (none) -> 10uF for dev; PD (none) -> CAP CER 10UF 25V X5R 0603
- C6, C7, C82, C9: MPN (none) -> GRT188R61E106ME13D; PD (none) -> CAP CER 10UF 25V X5R 0603
- C94: MPN (none) -> MSAST168BB5475MTNA01; PD (none) -> CAP CER 4.7UF 25V X5R 0603
- C96, C97: MPN (none) -> GRT188R61E225ME13D; PD (none) -> CAP CER 2.2UF 25V X5R 0603
- D1: value SMBJ13A -> SMBJ12A; MPN SMBJ13A -> SMBJ12A; PD (none) -> TVS DIODE 12VWM 19.9VC DO214AA
- D13: value SMAJ13A -> SMBJ12A; MPN SMAJ13A -> SMBJ12A; PD (none) -> TVS DIODE 12VWM 19.9VC DO214AA
- D14, D15, D5, D6: MPN XL-1608PGC-06 -> 150060GS75000; PD CHIP LED 0603 GREEN SMD -> LED GREEN CLEAR 0603 SMD
- D2: MPN (none) -> 150060GS75000; PD (none) -> LED GREEN CLEAR 0603 SMD
- D3: PD (none) -> DIODE SCHOTTKY 40V 1A SOD123W
- D4: MPN (none) -> BZT52C15; PD (none) -> DIODE ZENER 15V 500MW SOD123
- J1: footprint Connector_Molex:Molex_Pico-Lock_504050-0691_1x06-1MP_P1.50mm_Horizontal -> CustomFootprints:Molex_Pico-Lock_504050-0691_1x06-1MP_P1.50mm_Horizontal; PD (none) -> CONN HEADER SMD R/A 6POS 1.5MM
- J10, J7, J9: MPN (none) -> 61304021121; PD (none) -> CONN HEADER VERT 40POS 2.54MM
- J4: footprint Connector_USB:USB_C_Receptacle_HCTL_HC-TYPE-C-16P-01A -> Connector_USB:USB_C_Receptacle_GCT_USB4105-xx-A_16P_TopMnt_Horizontal; MPN (none) -> USB4105-GF-A; PD (none) -> CONN RCP USB2.0 TYP C 16P SMD RA
- J5, J6: MPN (none) -> 0532610471; PD (none) -> CONN HEADER SMD R/A 4POS 1.25MM
- J8: MPN (none) -> 61304011121; PD (none) -> CONN HEADER VERT 40POS 2.54MM
- Q1: footprint CustomFootprints:PowerPAK-SO-8L_Option-2_VIS -> PowerPAK-SO-8L_Option-2_VIS; MPN (none) -> SQJ407EP-T1_GE3; PD (none) -> MOSFET P-CH 30V 60A PPAK SO-8
- Q2, Q3: PD (none) -> MOSFET P-CH 20V 4.2A SOT23
- Q4: MPN (none) -> DMG2302UK-7; PD (none) -> MOSFET N-CH 20V 2.8A SOT23
- R1, R4: MPN (none) -> ERJ-3EKF5101V; PD (none) -> RES SMD 5.1K OHM 1% 1/10W 0603
- R11, R83, R84, R85, R86: MPN (none) -> ERJ-3GEY0R00V; PD (none) -> RES SMD 0 OHM JUMPER 1/10W 0603
- R12, R69: MPN (none) -> ERJ-3EKF1004V; PD (none) -> RES SMD 1M OHM 1% 1/10W 0603
- R13, R59, R60, R61, R66, R67, R7: MPN (none) -> ERJ-3EKF1002V; PD (none) -> RES SMD 10K OHM 1% 1/10W 0603
- R2: MPN (none) -> ERJ-3EKF8663V; PD (none) -> RES SMD 866K OHM 1% 1/10W 0603
- R3: MPN (none) -> ERJ-3EKF1503V; PD (none) -> RES SMD 150K OHM 1% 1/10W 0603
- R5: MPN (none) -> ERJ-3EKF5110V; PD (none) -> RES SMD 511 OHM 1% 1/10W 0603
- R51, R52, R57, R58: MPN (none) -> ERJ-3EKF4701V; PD (none) -> RES SMD 4.7K OHM 1% 1/10W 0603
- R6: MPN (none) -> ERJ-3EKF4700V; PD (none) -> RES SMD 470 OHM 1% 1/10W 0603
- R62, R63, R64, R65: MPN (none) -> ERJ-3EKF33R0V; PD (none) -> RES SMD 33 OHM 1% 1/10W 0603
- R68, R70, R8: MPN (none) -> ERJ-3EKF1003V; PD (none) -> RES SMD 100K OHM 1% 1/10W 0603
- R79, R80: MPN (none) -> ERJ-3EKF1801V; PD (none) -> RES SMD 1.8K OHM 1% 1/10W 0603
- R81, R82: MPN (none) -> ERJ-3EKF1000V; PD (none) -> RES SMD 100 OHM 1% 1/10W 0603
- SW1: MPN (none) -> B3U-1000P; PD (none) -> SWITCH TACTILE SPST-NO 0.05A 12V
- U1: footprint CustomFootprints:DSG0008A -> DSG0008A; PD (none) -> IC ELECTRONIC FUSE 7.5% 8WSON
- U11: MPN (none) -> AP2112K-3.3TRG1; PD (none) -> IC REG LINEAR 3.3V 600MA SOT-25
- U13: footprint Package_SON:WSON-8-1EP_8x6mm_P1.27mm_EP3.4x4.3mm -> MT29F1G01ABAFDWB-IT_F:SON127P600X800X65-8N; PD (none) -> IC FLASH 1GBIT SPI 8UPDFN
- U14: MPN (none) -> MB85RS256BPNF-G-AMERE2; PD (none) -> IC FRAM 256KBIT SPI 8-SOP
- U2: MPN (none) -> USBLC6-2SC6; PD (none) -> TVS DIODE 5.25VWM 17VC SOT23-6
- U3: MPN (none) -> STM32H7A3VIT6; PD (none) -> IC MCU 32BIT 2MB FLASH 100LQFP
- Y1: MPN (none) -> ABM8G-24.000MHZ-18-D2Y-T3; PD (none) -> CRYSTAL 24.0000MHZ 18PF SMD
Other:
- note added: "CHANGE FP AWAY FROM SOD-123W"
- note added: "PLACEHOLDER W 10UF FOR DEV"

Commit message: updated the last few component symbols/fps, none very significant
Parts:
- Q1: footprint PowerPAK-SO-8L_Option-2_VIS -> CustomFootprints:PowerPAK-SO-8L_Option-2_VIS
- U1: footprint DSG0008A -> CustomFootprints:DSG0008A
Changed lines of the file:
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@@
 			)
 		)
-		(property "Footprint" "PowerPAK-SO-8L_Option-2_VIS"
+		(property "Footprint" "CustomFootprints:PowerPAK-SO-8L_Option-2_VIS"
 			(at 111.76 30.48 0)
 			(effects
@@
 			)
 		)
-		(property "Footprint" "DSG0008A"
+		(property "Footprint" "CustomFootprints:DSG0008A"
 			(at 75.184 59.182 0)
 			(effects
